File: LRC-0/_restore_backup_2026-08-11T08-04-35-821/LRC-0.kicad_sch (KiCad schematic)
At the start: 57 parts, among them J1 USB_C_Receptacle_USB2.0_14P, J2 Battery, J3 SMA, J4 u.FL, J5 Conn_01x08, SW1 EN, SW2 BOOT, U2 AP7361C-33E, U3 TVS1400DRV, U4 BQ24075RGT, U5 ESP32-C6-MINI-1, U6 SX1262IMLTRT, U7 BGS12WN6E6327, U8 BGS12WN6E6327, Y1 TX32-33015S-32.000-X-R

Commit message: minor fixes to kicad version history
Parts:
- added R10: 10k, Resistor_SMD:R_0402_1005Metric, symbol Device:R
Connections:
- net +3V3: now also R10.1
- net RF1: now also FL1.8 (SW_RFO); no longer FL1.6 (SW_RFI), U8.3 (RF1)
- net RF2: now also FL1.6 (SW_RFI); no longer FL1.8 (SW_RFO), U8.1 (RF2)
- net IO8: no longer names the net of U5.22 (IO8)
- net IO8: now also R10.2
- new net SW_RFI: U8.3 (RF1)
- new net SW_RFO: U8.1 (RF2)
