File: LRC-0/PLOT/LRC-0.kicad_sch (KiCad schematic)
At the start: 69 parts, among them J1 USB_C_Receptacle_USB2.0_14P, J2 Battery, J3 Conn_01x10, J4 SMA, J5 u.FL, SW1 EN, SW2 BOOT, U1 AP7361C-33E, U2 TVS1400DRV, U3 BQ24075RGT, U4 ESP32-C6-MINI-1, U5 SX1262IMLTRT, U6 4259-63, U8 4259-63, Y1 TX32-33015S-32.000-X-R

Commit message: file organization
Parts:
- removed H1, H2, H3, H4: MountingHole, MountingHole:MountingHole_2.2mm_M2, symbol Mechanical:MountingHole
- added H1, H2, H3, H4: MountingHole_Pad, MountingHole:MountingHole_3.2mm_M3, symbol Mechanical:MountingHole_Pad
- added J6: USB_C_Receptacle_USB2.0_16P, symbol Connector:USB_C_Receptacle_USB2.0_16P
- C12, R14: now left out of the parts list
- C14, C16, C21, C23, C24, C27, J3, L3, L4: now not fitted
Connections:
- net GND: now also H1.1, H2.1, H3.1, H4.1
- new net: J6.A1 (GND), J6.A12 (GND), J6.B1 (GND), J6.B12 (GND)
- new net: J6.A4 (VBUS), J6.A9 (VBUS), J6.B4 (VBUS), J6.B9 (VBUS)
