File: LRC-0/_restore_backup_2026-08-31T16-39-55-173/LRC-0.kicad_pcb (KiCad board)
At the start: 4 copper layers, 46 x 40 mm, 59 parts, among them J1 USB_C_Receptacle_USB2.0_14P, J2 Battery, J3 Conn_01x04, J4 u.FL, J5 u.FL, J6 Conn_01x08, SW1 EN, SW2 BOOT, SW3 SW_SPDT, U1 AP7361C-33E, U2 TVS1400DRV, U3 BQ24075RGT, U4 ESP32-C6-MINI-1, U5 SX1262IMLTRT, U6 4259-63, U8 4259-63, Y1 TX32-33015S-32.000-X-R

Commit message: fixes idk
Parts:
- removed J6: Conn_01x08, Connector_JST:JST_PHD_S8B-PHDSS_2x04_P2.00mm_Horizontal
- added G***: LOGO, LOGO, B.Cu at (32.2, 11.0)
- added R16: 10k, Resistor_SMD:R_0402_1005Metric, F.Cu at (0.95, 0.49)
- J3: value Conn_01x04 -> Conn_01x08; footprint Connector_PinHeader_1.00mm:PinHeader_2x02_P1.00mm_Vertical -> Connector_JST:JST_PHD_S8B-PHDSS_2x04_P2.00mm_Horizontal
- moved J3 24.0 mm to (10.5, 34.4)
Connections:
- J3 pad 3: /SDA -> /SCK
- J3 pad 4: /SCL -> /MOSI
- U4 pad 16: /DSS -> /CS
- U4 pad 5: /SCL -> unconnected-(U4-IO2-Pad5)
- U4 pad 6: /SDA -> unconnected-(U4-IO3-Pad6)
Routing:
- net /DSS: track 15.8 -> 0.00 mm, vias 1 -> 0
- net /CS: track 0.00 -> 15.8 mm, vias 0 -> 1
- net /SCL: track 10.3 -> 0.00 mm, vias 1 -> 0
- net /SDA: track 8.03 -> 0.00 mm, vias 1 -> 0
- net +3V3: track 22.4 -> 17.8 mm
- net GND: vias 756 -> 765
