File: LRC-0/_restore_backup_2026-08-31T16-39-55-173/LRC-0.kicad_sch (KiCad schematic)
At the start: 71 parts, among them J1 USB_C_Receptacle_USB2.0_14P, J2 Battery, J3 Conn_01x04, J4 u.FL, J5 u.FL, J6 Conn_01x08, SW1 EN, SW2 BOOT, SW3 SW_SPDT, U1 AP7361C-33E, U2 TVS1400DRV, U3 BQ24075RGT, U4 ESP32-C6-MINI-1, U5 SX1262IMLTRT, U6 4259-63, U8 4259-63, Y1 TX32-33015S-32.000-X-R

Commit message: fixes idk
Parts:
- removed J3: Conn_01x04, Connector_PinHeader_1.00mm:PinHeader_2x02_P1.00mm_Vertical, symbol Connector_Generic:Conn_01x04
- removed J6: Conn_01x08, Connector_JST:JST_PHD_S8B-PHDSS_2x04_P2.00mm_Horizontal, symbol Connector_Generic:Conn_01x08
- added D3: LED, symbol Device:LED
- added J3: Conn_01x08, Connector_JST:JST_PHD_S8B-PHDSS_2x04_P2.00mm_Horizontal, symbol Connector_Generic:Conn_01x08
- added R16: 10k, Resistor_SMD:R_0402_1005Metric, symbol Device:R
Connections:
- net +3V3: now also J3.2 (Pin_2)
- net BLK: now also J3.8 (Pin_8)
- net DC: now also J3.6 (Pin_6)
- net GND: now also D3.1 (K), J3.1 (Pin_1)
- net MOSI: now also J3.4 (Pin_4)
- net RST: now also J3.5 (Pin_5)
- net SCK: now also J3.3 (Pin_3)
- net DSS renamed CS
- net CS: now also J3.7 (Pin_7)
- net SCL: no longer names the net of U4.5 (IO2)
- net SDA: no longer names the net of U4.6 (IO3)
- new net: D3.2 (A), R16.2
- new net TRX_IND: R16.1
