File: LRC-0/LRC-0.kicad_pcb (KiCad board)
At the start: 4 copper layers, 46 x 40 mm, 59 parts, among them J1 USB_C_Receptacle_USB2.0_14P, J2 Battery, J3 Conn_01x04, J4 u.FL, J5 u.FL, J6 Conn_01x08, SW1 EN, SW2 BOOT, SW3 SW_SPDT, U1 AP7361C-33E, U2 TVS1400DRV, U3 BQ24075RGT, U4 ESP32-C6-MINI-1, U5 SX1262IMLTRT, U6 4259-63, U8 4259-63, Y1 TX32-33015S-32.000-X-R

Commit message: final fixes
Parts:
- removed U1: AP7361C-33E, Package_TO_SOT_SMD:SOT-223-3_TabPin2
- C1, C2, C4, C6, C7, C8: footprint Capacitor_SMD:C_0402_1005Metric -> Capacitor_SMD:C_0603_1608Metric
- H1, H2, H3, H4: value MountingHole_Pad_MP -> MountingHole; footprint MountingHole:MountingHole_2.2mm_M2_Pad_TopOnly -> MountingHole:MountingHole_2.2mm_M2
- J3: footprint Connector_PinHeader_1.00mm:PinHeader_2x02_P1.00mm_Vertical -> Connector_PinHeader_2.54mm:PinHeader_2x02_P2.54mm_Vertical
- J4, J5: footprint Connector_Coaxial:U.FL_Hirose_U.FL-R-SMT-1_Vertical -> Connector_Coaxial:SMA_BAT_Wireless_BWSMA-KWE-Z001
- moved H3 34.0 mm to (43.0, 37.0)
- moved H4 34.0 mm to (43.0, 3.00)
- moved SW3 3.08 mm to (22.3, 10.5)
- moved C7 1.78 mm to (28.5, 11.2)
- moved J3 1.37 mm to (34.8, 36.5), turned to 90 degrees
- moved C1 1.23 mm to (18.8, 14.5), turned to 90 degrees
- moved R5 1.09 mm to (30.3, 11.8)
- moved D1 1.09 mm to (30.6, 3.40), turned to 0 degrees
- moved R9 1.06 mm to (33.1, 5.40), turned to 90 degrees
- moved D2 0.71 mm to (34.1, 3.40), turned to 180 degrees
- moved C6 0.64 mm to (31.6, 7.10)
- moved C4 0.51 mm to (31.6, 13.2)
- moved J6 0.38 mm to (10.5, 34.8)
- moved R10 0.37 mm to (31.5, 5.40)
- moved C2 0.22 mm to (18.8, 17.5)
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Connections:
- U4 pad 5: /SCL -> /SDA
- U4 pad 6: /SDA -> /SCL
Routing:
- net +3V3: track 22.4 -> 28.6 mm
- net VOUT: track 12.4 -> 17.4 mm
- net VCC: track 18.6 -> 23.3 mm, vias 2 -> 3
- net /SDA: track 8.03 -> 11.0 mm
- net GND: track 19.9 -> 17.7 mm, vias 756 -> 695
- net /ANT2: track 4.21 -> 5.74 mm
- net /SCL: track 10.3 -> 8.94 mm
- net /ANT1: track 5.48 -> 6.82 mm
- net Net-(U3-ILIM): track 2.41 -> 1.23 mm
- net Net-(D2-K): track 7.20 -> 6.24 mm
- removed copper zone on F.Cu, net VCC
Other:
- outline, holes or cut-outs redrawn

Commit message: something
Parts:
- added U1: AP7361C-33E, Package_TO_SOT_SMD:SOT-223-3_TabPin2, F.Cu at (24.9, 16.4)
- moved C2 1.03 mm to (19.7, 16.9)
- moved C1 1.03 mm to (19.7, 13.9)
Connections:
- net /BLK renamed /B_{d}
- J6 pad 1: GND -> +3V3
- J6 pad 2: +3V3 -> GND
Routing:
- net +3V3: track 28.6 -> 27.5 mm
- net VOUT: track 17.4 -> 18.2 mm
- net VCC: vias 3 -> 2
- net GND: vias 695 -> 692

Commit message: via fixes
Routing:
- net GND: vias 692 -> 691
